File: ODRIVE_V2.0.kicad_sch (KiCad schematic)
At the start: 31 parts, among them J1 Jack-DC, J2 USB_B, J3 Conn_01x04_Pin, J9 Conn_01x04_Pin, U1 L7805, U1 TJA1050T_CM_118, U3 CH340G, U5 LM2596S-5, Y1 Crystal

Commit message: first add1
Parts:
- removed C?: 47uF, Capacitor_THT:C_Radial_D6.3mm_H11.0mm_P2.50mm, symbol Device:C_Small
- removed C?: 10uF, Capacitor_THT:C_Radial_D6.3mm_H11.0mm_P2.50mm, symbol Device:C_Small
- removed U1: L7805, Package_TO_SOT_THT:TO-220-3_Vertical, symbol Regulator_Linear:L7805
- added R2 (x2): R, Resistor_THT:R_Axial_DIN0204_L3.6mm_D1.6mm_P7.62mm_Horizontal, symbol Device:R
Connections:
- net GND: now also D4.2 (A), U5.3 (GND), U5.5 (~{ON}/OFF), R2.2
- net VCC: now also L1.2, R2.2
- net VDD: now also U5.1 (VIN)
- net at L1.1: now also D4.1 (K), U5.2 (OUT)
- net at U5.4 (FB): now also R2.1, R2.1
Other:
- moved on the sheet: D4, L1
